Commit message: removed 2 extra cameras

File: hector_quadrotor/hector_quadrotor_description/urdf/quadrotor_velodyne.urdf.xacro (robot description, xacro)
@@ -20,13 +20,3 @@
       <origin xyz="0.05 0.0 -0.06" rpy="0 0.43 0"/>
     </xacro:generic_camera>
-    <!-- Backward facing camera -->
-    <xacro:include filename="$(find hector_sensors_description)/urdf/generic_camera.urdf.xacro" />
-    <xacro:generic_camera name="bottom_cam" parent="base_link" ros_topic="camera/image" cam_info_topic="camera/camera_info" update_rate="10" res_x="512" res_y="512" image_format="R8G8B8" hfov="90">
-      <origin xyz="0 0.0 -0.09" rpy="0 ${M_PI_2} 0"/>
-    </xacro:generic_camera>
-    <!-- Asus Xiton Live Pro -->
-    <xacro:include filename="$(find hector_sensors_description)/urdf/asus_camera.urdf.xacro" />
-    <xacro:asus_camera name="camera" parent="base_link">
-      <origin xyz="0.1 0.0 -0.03" rpy="0 0 0"/>
-    </xacro:asus_camera>
 </robot>
